File: OnePress schematic.kicad_sch (KiCad schematic)
At the start: 1 part, among them U1 Arduino_Pro_Micro

Commit message: test
Parts:
- added R1: Resistor, symbol ScottoKeebs:Placeholder_Resistor
Changed lines of the file:
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@@
 (kicad_sch
-	(version 20231120)
+	(version 20260306)
 	(generator "eeschema")
-	(generator_version "8.0")
+	(generator_version "10.0")
 	(paper "A4")
+	(symbol
+		(lib_id "ScottoKeebs:Placeholder_Resistor")
+		(at 133.35 114.3 0)
+		(unit 1)
+		(body_style 1)
+		(exclude_from_sim no)
+		(in_bom yes)
+		(on_board yes)
+		(in_pos_files yes)
+		(dnp no)
+		(fields_autoplaced yes)
+		(property "Reference" "R1"
+			(at 133.35 107.95 0)
+			(show_name no)
+			(do_not_autoplace no)
+			(effects
+				(font
+					(size 1.27 1.27)
+				)
+			)
+		)
+		(property "Value" "Resistor"
+			(at 133.35 110.49 0)
+			(show_name no)
+			(do_not_autoplace no)
+			(effects
+				(font
+					(size 1.27 1.27)
+				)
+			)
+		)
+		(property "Footprint" ""
+			(at 133.35 116.078 0)
+			(hide yes)
+			(show_name no)
+			(do_not_autoplace no)
+			(effects
+				(font
+					(size 1.27 1.27)
+				)
+			)
+		)
+		(property "Datasheet" ""
+			(at 133.35 114.3 90)
+			(hide yes)
+			(show_name no)
+			(do_not_autoplace no)
+			(effects
+				(font
+					(size 1.27 1.27)
+				)
+			)
+		)
+		(property "Description" "Resistor"
+			(at 133.35 114.3 0)
+			(hide yes)
+			(show_name no)
+			(do_not_autoplace no)
+			(effects
+				(font
+					(size 1.27 1.27)
+				)
+			)
+		)
+		(pin "2"
+		)
+		(pin "1"
+		)
+		(instances
+			(project "OnePress schematic"
+				(path "/0ba40caf-3b9c-413a-892d-6c35d33f7fe3"
+					(reference "R1")
+					(unit 1)
+				)
+			)
+		)
+	)
 	(symbol
 		(lib_id "ScottoKeebs:MCU_Arduino_Pro_Micro")
 		(at 82.55 105.41 0)
 		(unit 1)
+		(body_style 1)
 		(exclude_from_sim no)
 		(in_bom yes)
 		(on_board yes)
+		(in_pos_files yes)
 		(dnp no)
 		(fields_autoplaced yes)
 		(property "Reference" "U1"
 			(at 82.55 83.82 0)
+			(show_name no)
+			(do_not_autoplace no)
 			(effects
 				(font
@@
 		(property "Value" "Arduino_Pro_Micro"
 			(at 82.55 86.36 0)
+			(show_name no)
+			(do_not_autoplace no)
 			(effects
 				(font
@@
 		(property "Footprint" "ScottoKeebs_MCU:Arduino_Pro_Micro"
 			(at 82.55 128.27 0)
-			(effects
-				(font
-					(size 1.524 1.524)
-				)
-				(hide yes)
+			(hide yes)
+			(show_name no)
+			(do_not_autoplace no)
+			(effects
+				(font
+					(size 1.524 1.524)
+				)
 			)
 		)
 		(property "Datasheet" ""
 			(at 109.22 168.91 90)
-			(effects
-				(font
-					(size 1.524 1.524)
-				)
-				(hide yes)
+			(hide yes)
+			(show_name no)
+			(do_not_autoplace no)
+			(effects
+				(font
+					(size 1.524 1.524)
+				)
 			)
 		)
 		(property "Description" ""
 			(at 82.55 105.41 0)
-			(effects
-				(font
-					(size 1.27 1.27)
-				)
-				(hide yes)
+			(hide yes)
+			(show_name no)
+			(do_not_autoplace no)
+			(effects
+				(font
+					(size 1.27 1.27)
+				)
 			)
 		)
@@
 		)
 	)
+	(embedded_fonts no)
 )

Commit message: test
Parts:
- removed R1: Resistor, symbol ScottoKeebs:Placeholder_Resistor
- removed U1: Arduino_Pro_Micro, ScottoKeebs_MCU:Arduino_Pro_Micro, symbol ScottoKeebs:MCU_Arduino_Pro_Micro
- added D1, D2, D3, D4, D5, D6, D7, D8, D9: (no value), ScottoKeebs_Components:Diode_DO-35, symbol ScottoKeebs:Placeholder_Diode
- added D10, D11, D12: D_Capacitance, Capacitor_SMD:C_01005_0402Metric, symbol Device:D_Capacitance
- added LS1: Speaker, Buzzer_Beeper:Speaker_CUI_CMR-1206S-67, symbol Device:Speaker
- added MK1: Microphone, Sensor_Audio:CUI_CMC-4013-SMT, symbol Device:Microphone
- added Q1: 2N2219, Package_TO_SOT_THT:TO-39-3, symbol Transistor_BJT:2N2219
- added R2: 1000, Resistor_SMD:R_01005_0402Metric, symbol Device:R
- added R3: 2.2 k, Resistor_SMD:R_01005_0402Metric, symbol Device:R
- added R4, R5, R6: R, Resistor_SMD:R_01005_0402Metric, symbol Device:R
- added S1, S2, S3, S4, S5, S6, S7, S8, S9: (no value), ScottoKeebs_MX:MX_PCB_1.00u, symbol ScottoKeebs:Placeholder_Keyswitch
- added U2: Arduino_Pro_Micro, ScottoKeebs_MCU:Arduino_Pro_Micro, symbol ScottoKeebs:MCU_Arduino_Pro_Micro
- added U3: SSM2167, Package_SO:MSOP-10_3x3mm_P0.5mm, symbol Amplifier_Audio:SSM2167
Connections:
- new net: D4.2 (A), S4.2
- new net: D2.2 (A), S2.2
- new net: D11.2 (A), U3.6 (AVG)
- new net: D6.2 (A), S6.2
- new net: D7.2 (A), S7.2
- new net: D12.1 (K), U3.2 (VCAIN)
- new net: D12.2 (A), U3.4 (BUFOUT)
- new net: LS1.2, Q1.3 (C)
- new net: D9.2 (A), S9.2
- new net: Q1.1 (E), U2.3 (GND)
- new net: Q1.2 (B), R2.1
- new net: D10.1 (K), MK1.2 (+), R3.2
- new net: D5.2 (A), S5.2
- new net: R5.1, U3.8 (COMP)
- new net: R4.1, U3.3 (~{SD})
- new net: R2.2, U2.12 (9/PB5)
- new net: D10.2 (A), U3.5 (IN+)
- new net: D1.2 (A), S1.2
- new net: D3.2 (A), S3.2
- new net: R6.2, U3.7 (GATE)
- new net: D8.2 (A), S8.2
- new net Column 0: S1.1, S4.1, S7.1, U2.5 (2/PD1)
- new net Column 1: S2.1, S5.1, S8.1, U2.6 (3/PD0)
- new net Column 3: S3.1, S6.1, S9.1, U2.7 (4/PD4)
- new net GNDS: D11.1 (K), MK1.1 (-), U2.23 (GND), U2.4 (GND), U3.1 (GND)
- new net Row 0: D1.1 (K), D2.1 (K), D3.1 (K), U2.8 (5/PC6)
- new net Row 1: D4.1 (K), D5.1 (K), D6.1 (K), U2.9 (6/PD7)
- new net Row 2: D7.1 (K), D8.1 (K), D9.1 (K), U2.10 (7/PE6)
- new net VA3: U2.20 (A3/PF4), U3.9 (VOUT)
- new net VCC: LS1.1, R3.1, R4.2, R5.2, R6.1, U2.21 (VCC), U3.10 (V+)
